File: panel16x16/panel16x16.kicad_pcb (KiCad board)
At the start: 4 copper layers, 50 x 50 mm, 348 parts, among them Q1 DMG2301L, Q10 DMG2301L, Q11 DMG2301L, Q12 DMG2301L, Q13 DMG2301L, Q14 DMG2301L, Q15 DMG2301L, Q16 DMG2301L, Q2 DMG2301L, Q3 DMG2301L, Q4 DMG2301L, Q5 DMG2301L, Q6 DMG2301L, Q7 DMG2301L, Q8 DMG2301L, Q9 DMG2301L, U1 74HC595, U2 74HC595, U3 74HC595, U4 74HC595, U5 74HC595, U6 74HC595, U7 74HC595, U8 74HC595, U9 74LVC2G17

Commit message: Finish PCB design
Parts:
- removed C9: 100nF, Capacitor_SMD:C_0603_1608Metric
- removed JGND2, JPWR2, JRCLK2, JSCLK2: Conn_01x01, TestPoint:TestPoint_Pad_2.0x2.0mm
- JGND1, JPWR1, JRCLK1, JSCLK1, JSERIN1, JSEROUT1, Q1, Q10, Q11, Q12, Q13, Q14, Q15, Q16, Q2, Q3, Q4, Q5, Q6, Q7, Q8, Q9, U7, U8, U9: moved to B.Cu
- moved JSEROUT1 189.5 mm to (50.2, 75.0), turned to 180 degrees
- moved Q8 188.7 mm to (61.5, 69.6), turned to -90 degrees
- moved Q7 184.1 mm to (64.9, 69.6), turned to -90 degrees
- moved Q1 183.1 mm to (61.7, 58.1), turned to 90 degrees
- moved Q2 181.4 mm to (65.2, 58.1), turned to 90 degrees
- moved Q3 179.8 mm to (68.6, 58.1), turned to 90 degrees
- moved Q4 179.7 mm to (68.9, 62.1)
- moved Q6 179.5 mm to (68.3, 69.6), turned to -90 degrees
- moved Q5 178.8 mm to (68.9, 65.6)
- moved C7 178.2 mm to (57.3, 59.5), turned to 0 degrees
- moved RB1 175.8 mm to (51.8, 90.6), turned to 0 degrees
- moved Q16 175.1 mm to (80.0, 89.0), turned to 90 degrees
- moved Q15 170.8 mm to (83.4, 89.0), turned to 90 degrees
- moved Q9 170.1 mm to (80.0, 76.5), turned to 90 degrees
- moved Q10 167.9 mm to (83.4, 76.5), turned to 90 degrees
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Connections:
- U1 pad 9: Net-(JSEROUT1-Pin_1) -> Net-(U1-QH')
- U6 pad 14: Net-(U6-SER) -> Net-(JSERIN1-Pin_1)
- U7 pad 9: Net-(U6-SER) -> Net-(JSEROUT1-Pin_1)
- U8 pad 14: Net-(JSERIN1-Pin_1) -> Net-(U1-QH')
Routing:
- net /SCLK: track 0.00 -> 130.4 mm, vias 0 -> 11
- net /RCLK: track 0.00 -> 123.7 mm, vias 0 -> 2
- net VCC: track 0.00 -> 99.7 mm, vias 0 -> 28
- net GND: track 13.0 -> 92.6 mm, vias 6 -> 14
- net Net-(U7-SER): track 0.00 -> 53.4 mm, vias 0 -> 2
- net Net-(JSEROUT1-Pin_1): track 0.00 -> 43.6 mm, vias 0 -> 2
- net Net-(JSERIN1-Pin_1): track 0.00 -> 26.8 mm, vias 0 -> 2
- net Net-(U1-QH'): track 0.00 -> 23.8 mm, vias 0 -> 2
- net Net-(U3-SER): track 0.00 -> 22.0 mm
- net Net-(U3-QA): track 0.00 -> 18.1 mm
- net Net-(U1-QA): track 0.00 -> 14.8 mm
- net Net-(U2-QB): track 0.00 -> 13.4 mm
- net Net-(U3-QG): track 0.00 -> 12.9 mm
- net Net-(U3-QD): track 0.00 -> 12.8 mm
- net Net-(Q13-G): track 0.00 -> 12.6 mm
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- added copper zone on In2.Cu, net VCC
