File: panel16x16/panel16x16.kicad_sch (KiCad schematic)
At the start: 348 parts, among them Q1 DMG2301L, Q10 DMG2301L, Q11 DMG2301L, Q12 DMG2301L, Q13 DMG2301L, Q14 DMG2301L, Q15 DMG2301L, Q16 DMG2301L, Q2 DMG2301L, Q3 DMG2301L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

Commit message: Finish PCB design
Parts:
- removed C9: 100nF, Capacitor_SMD:C_0603_1608Metric, symbol Device:C_Small
- removed JGND2, JPWR2, JRCLK2, JSCLK2: Conn_01x01, TestPoint:TestPoint_Pad_2.0x2.0mm, symbol Connector_Generic:Conn_01x01
Connections:
- net at U6.14 (SER): now also JSERIN1.1 (Pin_1); no longer U7.9 (QH')
- net at JSEROUT1.1 (Pin_1): now also U7.9 (QH'); no longer U1.9 (QH')
- net at U8.14 (SER): now also U1.9 (QH'); no longer JSERIN1.1 (Pin_1)
